File: Boards/V1-3/V1-3-1 (Double Stack)/Flodar_Board_V1-3-1.brd (EAGLE design)
At the start: 70 x 66 mm, 12 parts, among them U2 LP2981-33DBVR

Commit message: Update Flodar_Board_V1-3-1.brd
Parts:
- moved JP1 29.5 mm to (55.1, 18.0)
Routing:
- net 12V: track 35.7 -> 65.5 mm
Other:
- board text added: "FloDar Power & Breakout V1.3.1"
- board text removed: "FloDar Power & Breakout V1.2"
Changed lines of the file:
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@@
 <drawing>
 <settings>
-<setting alwaysvectorfont="yes"/>
+<setting alwaysvectorfont="no"/>
 <setting verticaltext="up"/>
 </settings>
@@
 <dimension x1="0" y1="72" x2="0" y2="6" x3="-2" y3="39" textsize="1.778" layer="1" dtype="diameter"/>
 <text x="9" y="66" size="1.778" layer="25">FloDar Power &amp; Breakout
-V1.2</text>
+V1.3.1</text>
 <dimension x1="5" y1="73.5" x2="69" y2="73.5" x3="37" y3="73.5" textsize="1.778" layer="1"/>
 <dimension x1="0" y1="69" x2="0" y2="9" x3="0" y3="39" textsize="1.778" layer="1"/>
-<text x="25" y="12" size="1.4224" layer="21" rot="R90">12V</text>
-<text x="27.5" y="11" size="1.4224" layer="21" rot="R90">GND</text>
+<text x="54.5" y="12" size="1.4224" layer="21" rot="R90">12V</text>
+<text x="57.5" y="11.5" size="1.4224" layer="21" rot="R90">GND</text>
 <text x="40" y="59" size="1.4224" layer="21" rot="R225">5V</text>
 <text x="43" y="59" size="1.4224" layer="21" rot="R225">GND</text>
@@
 <attribute name="VALUE" x="20.17" y="19.71" size="1.27" layer="27" rot="R90"/>
 </element>
-<element name="JP1" library="pinhead" library_urn="urn:adsk.eagle:library:325" package="1X02" package3d_urn="urn:adsk.eagle:package:22435/2" value="" x="25.612" y="17.328" smashed="yes">
-<attribute name="NAME" x="26.5042" y="20.8432" size="1.27" layer="25" ratio="10" rot="R180"/>
-<attribute name="POPULARITY" value="98" x="67.522" y="-14.422" size="1.778" layer="27" display="off"/>
-<attribute name="VALUE" x="23.072" y="14.153" size="1.27" layer="27"/>
+<element name="JP1" library="pinhead" library_urn="urn:adsk.eagle:library:325" package="1X02" package3d_urn="urn:adsk.eagle:package:22435/2" value="" x="55.112" y="17.955" smashed="yes">
+<attribute name="NAME" x="56.0042" y="21.4702" size="1.27" layer="25" ratio="10" rot="R180"/>
+<attribute name="POPULARITY" value="98" x="97.022" y="-13.795" size="1.778" layer="27" display="off"/>
+<attribute name="VALUE" x="52.572" y="14.78" size="1.27" layer="27"/>
 </element>
 <element name="U2" library="LP2981-33DBVR" package="SOT95P280X145-5N" value="LP2981-33DBVR" x="15.14" y="17.29" smashed="yes" rot="R90">
@@
 <via x="59" y="25" extent="1-16" drill="0.35"/>
 <via x="25" y="36.5" extent="1-16" drill="0.35"/>
-<via x="33.5" y="13" extent="1-16" drill="0.35"/>
-<via x="35.5" y="17" extent="1-16" drill="0.35"/>
+<via x="33.5" y="13.5" extent="1-16" drill="0.35"/>
+<via x="35.5" y="16.5" extent="1-16" drill="0.35"/>
 <via x="19" y="42" extent="1-16" drill="0.35"/>
 <via x="15.5" y="45" extent="1-16" drill="0.35"/>
@@
 <contactref element="U2" pad="3"/>
 <contactref element="U$1" pad="HVIN"/>
-<wire x1="16.09" y1="16.035" x2="23.049" y2="16.035" width="0.508" layer="1"/>
-<wire x1="23.049" y1="16.035" x2="24.342" y2="17.328" width="0.508" layer="1"/>
 <wire x1="14.19" y1="16.035" x2="14.19" y2="13.17" width="0.508" layer="1"/>
 <wire x1="14.19" y1="13.17" x2="14.04" y2="13.02" width="0.508" layer="1"/>
@@
 <wire x1="14.04" y1="13.02" x2="16.09" y2="15.07" width="0.508" layer="1"/>
 <wire x1="16.09" y1="15.07" x2="16.09" y2="16.035" width="0.508" layer="1"/>
+<wire x1="16.09" y1="16.035" x2="16.125" y2="16" width="0.508" layer="1"/>
+<wire x1="32.5" y1="16" x2="34.5" y2="18" width="0.508" layer="1"/>
+<wire x1="34.5" y1="18" x2="53.797" y2="18" width="0.508" layer="1"/>
+<wire x1="53.797" y1="18" x2="53.842" y2="17.955" width="0.508" layer="1"/>
+<wire x1="16.125" y1="16" x2="32.5" y2="16" width="0.508" layer="1"/>
 </signal>
 <signal name="USB">
